File: _autosave-keeb-PCB1.kicad_sch (KiCad schematic)
At the start: 14 parts, among them SW1 SW_Push, U1 ATmega32U4-A, Y1 16MHz

Commit message: Update _autosave-keeb-PCB1.kicad_sch
Parts:
- added J1: AVR-ISP-6, symbol Connector:AVR-ISP-6
- added USB1: Molex-0548190589, symbol random-keyboard-parts:Molex-0548190589
Connections:
- net +5V: now also J1.2 (VCC)
- net GND: now also J1.6 (GND)
- net D-: now reaches R3.1
- net D+: now reaches R2.1
- net MOSI: now reaches U1.10 (PB2)
- net MOSI: now also J1.4 (MOSI)
- net MISO: now reaches U1.11 (PB3)
- net MISO: now also J1.1 (MISO)
- net SCK: now reaches U1.9 (PB1)
- net SCK: now also J1.3 (SCK)
- new net RESET: J1.5 (~{RST})
Other:
- moved on the sheet: C2, C3, C4, C5
